File: SisCoCaf/SisCoCaf.sch (KiCad schematic (older format))
At the start: 20 parts

Commit message: Listo para revisión del esquemático
Parts:
- gave numbers to parts that had none: 10
- renumbered R5 to R4, R8 to R5, R4 to R7, R7 to R8
Connections:
- no-connect marks 0 -> 13
Other:
- note added: "Caracteristicas técnicas:"
- note added: "Fuente de Alimentación"
- note added: "PCB:\n- De 1 capa.\n- Se utilizará técnica de planchado.\n- Material: Fibra de vidrio.\n- Color: Verde.\n\nEntorno:\n- Temperatura de trabajo: -25ºC a +85ºC\n\nElectrónica:\nCorriente: 500 miliamperios.\nVoltaje: 12Vts. DC\n\n"

Commit message: Agrego huellas
Parts:
- BZ1: footprint (none) -> Buzzer_Beeper:Buzzer_12x9.5RM7.6
- D1: footprint (none) -> LED_THT:LED_D3.0mm
- IC1: footprint (none) -> Package_DIP:DIP-28_W15.24mm_Socket
- J1, J2: footprint (none) -> Connector_PinSocket_1.27mm:PinSocket_1x02_P1.27mm_Vertical
- J3, J4: footprint (none) -> Connector_PinHeader_1.00mm:PinHeader_1x03_P1.00mm_Vertical
- J5: footprint (none) -> Connector_PinHeader_1.00mm:PinHeader_1x02_P1.00mm_Vertical
- R1, R2, R3, R4, R5, R6, R7, R8: footprint (none) -> Resistor_THT:R_Axial_DIN0204_L3.6mm_D1.6mm_P7.62mm_Horizontal
Other:
- note added: "PCB:\n- De 1 capa.\n- Se utilizará técnica de planchado.\n- Material: Fibra de vidrio.\n- Color: Verde.\n\nEntorno:\n- Temperatura de trabajo: -25ºC a +85ºC\n\nElectrónica:\n- Corriente: 500 miliamperios.\n- Voltaje: 12Vts. DC"
- note removed: "PCB:\n- De 1 capa.\n- Se utilizará técnica de planchado.\n- Material: Fibra de vidrio.\n- Color: Verde.\n\nEntorno:\n- Temperatura de trabajo: -25ºC a +85ºC\n\nElectrónica:\nCorriente: 500 miliamperios.\nVoltaje: 12Vts. DC\n\n"
Changed lines of the file:
@@
 Title "SisCoCaf"
 Date "2018-09-08"
-Rev ""
+Rev "1.03"
 Comp "Roberto Compañy"
 Comment1 ""
@@
 F 0 "R1" H 2170 2146 50  0000 L CNN
 F 1 "1k" H 2170 2055 50  0000 L CNN
-F 2 "" V 2030 2100 50  0001 C CNN
+F 2 "Resistor_THT:R_Axial_DIN0204_L3.6mm_D1.6mm_P7.62mm_Horizontal" V 2030 2100 50  0001 C CNN
 F 3 "~" H 2100 2100 50  0001 C CNN
 	1    2100 2100
@@
 F 0 "R2" H 2820 2146 50  0000 L CNN
 F 1 "1k" H 2820 2055 50  0000 L CNN
-F 2 "" V 2680 2100 50  0001 C CNN
+F 2 "Resistor_THT:R_Axial_DIN0204_L3.6mm_D1.6mm_P7.62mm_Horizontal" V 2680 2100 50  0001 C CNN
 F 3 "~" H 2750 2100 50  0001 C CNN
 	1    2750 2100
@@
 F 0 "J2" H 10100 1300 50  0000 L CNN
 F 1 "Conn_01x02_Female" H 10077 1185 50  0000 L CNN
-F 2 "" H 10050 1300 50  0001 C CNN
+F 2 "Connector_PinSocket_1.27mm:PinSocket_1x02_P1.27mm_Vertical" H 10050 1300 50  0001 C CNN
 F 3 "~" H 10050 1300 50  0001 C CNN
 	1    10050 1300
@@
 F 0 "R3" H 7220 4996 50  0000 L CNN
 F 1 "5k6" H 7220 4905 50  0000 L CNN
-F 2 "" V 7080 4950 50  0001 C CNN
+F 2 "Resistor_THT:R_Axial_DIN0204_L3.6mm_D1.6mm_P7.62mm_Horizontal" V 7080 4950 50  0001 C CNN
 F 3 "~" H 7150 4950 50  0001 C CNN
 	1    7150 4950
@@
 F 0 "R7" V 9450 1600 50  0000 C CNN
 F 1 "220" V 9650 1600 50  0000 C CNN
-F 2 "" V 9480 1600 50  0001 C CNN
+F 2 "Resistor_THT:R_Axial_DIN0204_L3.6mm_D1.6mm_P7.62mm_Horizontal" V 9480 1600 50  0001 C CNN
 F 3 "~" H 9550 1600 50  0001 C CNN
 	1    9550 1600
@@
 F 0 "D1" H 9550 1750 50  0000 C CNN
 F 1 "LED" H 9550 1650 50  0000 C CNN
-F 2 "" H 9850 1750 50  0001 C CNN
+F 2 "LED_THT:LED_D3.0mm" H 9850 1750 50  0001 C CNN
 F 3 "~" H 9850 1750 50  0001 C CNN
 	1    9850 1750
@@
 F 0 "BZ1" H 10103 2979 50  0000 L CNN
 F 1 "Buzzer" H 10103 2888 50  0000 L CNN
-F 2 "" V 9925 3050 50  0001 C CNN
+F 2 "Buzzer_Beeper:Buzzer_12x9.5RM7.6" V 9925 3050 50  0001 C CNN
 F 3 "~" V 9925 3050 50  0001 C CNN
 	1    9950 2950
@@
 F 0 "R4" V 8943 3250 50  0000 C CNN
 F 1 "220" V 9034 3250 50  0000 C CNN
-F 2 "" V 9080 3250 50  0001 C CNN
+F 2 "Resistor_THT:R_Axial_DIN0204_L3.6mm_D1.6mm_P7.62mm_Horizontal" V 9080 3250 50  0001 C CNN
 F 3 "~" H 9150 3250 50  0001 C CNN
 	1    9150 3250
@@
 F 0 "J5" H 10023 4723 50  0000 R CNN
 F 1 "Conn_01x01_Male" H 10023 4632 50  0000 R CNN
-F 2 "" H 10050 4700 50  0001 C CNN
+F 2 "Connector_PinHeader_1.00mm:PinHeader_1x02_P1.00mm_Vertical" H 10050 4700 50  0001 C CNN
 F 3 "~" H 10050 4700 50  0001 C CNN
 	1    10050 4700
@@
 F 0 "R6" V 9193 4900 50  0000 C CNN
 F 1 "220" V 9284 4900 50  0000 C CNN
-F 2 "" V 9330 4900 50  0001 C CNN
+F 2 "Resistor_THT:R_Axial_DIN0204_L3.6mm_D1.6mm_P7.62mm_Horizontal" V 9330 4900 50  0001 C CNN
 F 3 "~" H 9400 4900 50  0001 C CNN
 	1    9400 4900
@@
 F 0 "J3" H 10023 2273 50  0000 R CNN
 F 1 "Conn_01x03_Male" H 10023 2182 50  0000 R CNN
-F 2 "" H 10050 2250 50  0001 C CNN
+F 2 "Connector_PinHeader_1.00mm:PinHeader_1x03_P1.00mm_Vertical" H 10050 2250 50  0001 C CNN
 F 3 "~" H 10050 2250 50  0001 C CNN
 	1    10050 2250
@@
 F 0 "J1" H 10100 900 50  0000 L CNN
 F 1 "Conn_01x02_Female" H 10077 785 50  0000 L CNN
-F 2 "" H 10050 900 50  0001 C CNN
+F 2 "Connector_PinSocket_1.27mm:PinSocket_1x02_P1.27mm_Vertical" H 10050 900 50  0001 C CNN
 F 3 "~" H 10050 900 50  0001 C CNN
 	1    10050 900
@@
 F 0 "R8" V 9600 900 50  0000 C CNN
 F 1 "220" V 9800 900 50  0000 C CNN
-F 2 "" V 9630 900 50  0001 C CNN
+F 2 "Resistor_THT:R_Axial_DIN0204_L3.6mm_D1.6mm_P7.62mm_Horizontal" V 9630 900 50  0001 C CNN
 F 3 "~" H 9700 900 50  0001 C CNN
 	1    9700 900
@@
 F 0 "R5" V 9200 1000 50  0000 C CNN
 F 1 "220" V 9450 1000 50  0000 C CNN
-F 2 "" V 9280 1000 50  0001 C CNN
+F 2 "Resistor_THT:R_Axial_DIN0204_L3.6mm_D1.6mm_P7.62mm_Horizontal" V 9280 1000 50  0001 C CNN
 F 3 "~" H 9350 1000 50  0001 C CNN
 	1    9350 1000
@@
 F 0 "IC1" H 6150 3837 60  0000 C CNN
 F 1 "LPC111X_102" H 6150 3731 60  0000 C CNN
-F 2 "" H 6150 2350 50  0001 C CNN
+F 2 "Package_DIP:DIP-28_W15.24mm_Socket" H 6150 2350 50  0001 C CNN
 F 3 "" H 6150 2350 50  0001 C CNN
 	1    6150 2350
@@
 F 0 "J4" H 10023 4023 50  0000 R CNN
 F 1 "Conn_01x03_Male" H 10023 3932 50  0000 R CNN
-F 2 "" H 10050 4000 50  0001 C CNN
+F 2 "Connector_PinHeader_1.00mm:PinHeader_1x03_P1.00mm_Vertical" H 10050 4000 50  0001 C CNN
 F 3 "~" H 10050 4000 50  0001 C CNN
 	1    10050 4000
@@
 Caracteristicas técnicas:
 Text Notes 1200 6500 0    79   ~ 0
-PCB:\n- De 1 capa.\n- Se utilizará técnica de planchado.\n- Material: Fibra de vidrio.\n- Color: Verde.\n\nEntorno:\n- Temperatura de trabajo: -25ºC a +85ºC\n\nElectrónica:\nCorriente: 500 miliamperios.\nVoltaje: 12Vts. DC\n\n
+PCB:\n- De 1 capa.\n- Se utilizará técnica de planchado.\n- Material: Fibra de vidrio.\n- Color: Verde.\n\nEntorno:\n- Temperatura de trabajo: -25ºC a +85ºC\n\nElectrónica:\n- Corriente: 500 miliamperios.\n- Voltaje: 12Vts. DC
 $EndSCHEMATC

Commit message: Esquemático corregido. PCB v1.0
Parts:
- removed J4: Conn_01x03_Male, Connector_PinHeader_1.00mm:PinHeader_1x03_P1.00mm_Vertical, symbol Connector:Conn_01x03_Male
- added BT1: Battery_Cell, Battery:BatteryHolder_Keystone_103_1x20mm, symbol Device:Battery_Cell
- added J1: Entrada, Connector_JST:JST_XH_B02B-XH-A_1x02_P2.50mm_Vertical, symbol Connector_Generic:Conn_01x02
- added J6: Conn_01x03_Male, Connector_JST:JST_XH_B03B-XH-A_1x03_P2.50mm_Vertical, symbol Connector:Conn_01x03_Male
- added JP1: Jumper, Connector_PinHeader_2.54mm:PinHeader_1x02_P2.54mm_Vertical, symbol Device:Jumper
- added MH1, MH2, MH3, MH4: MountingHole, MountingHole:MountingHole_2.2mm_M2, symbol Mechanical:MountingHole
- added R6, R7: 4k7, Resistor_THT:R_Axial_DIN0204_L3.6mm_D1.6mm_P7.62mm_Horizontal, symbol Device:R
- J2: footprint Connector_PinSocket_1.27mm:PinSocket_1x02_P1.27mm_Vertical -> Connector_PinSocket_2.54mm:PinSocket_1x02_P2.54mm_Vertical
- J4: renamed from J5; footprint Connector_PinHeader_1.00mm:PinHeader_1x02_P1.00mm_Vertical -> Connector_PinHeader_2.54mm:PinHeader_1x01_P2.54mm_Vertical
- J5: renamed from J3; footprint Connector_PinHeader_1.00mm:PinHeader_1x03_P1.00mm_Vertical -> Connector_JST:JST_XH_B03B-XH-A_1x03_P2.50mm_Vertical
- J7: renamed from J1; value Conn_01x02_Female -> Conn_01x02_Male; footprint Connector_PinSocket_1.27mm:PinSocket_1x02_P1.27mm_Vertical -> Connector_JST:JST_XH_B02B-XH-A_1x02_P2.50mm_Vertical
- Q1, Q2: footprint Package_TO_SOT_THT:TO-92_Inline -> Package_TO_SOT_THT:TO-92_HandSolder
- U1: footprint Package_TO_SOT_THT:TO-39-3 -> Package_TO_SOT_THT:TO-220-3_Vertical; symbol Regulator_Linear:LM317_TO39 -> Regulator_Linear:LM317L_TO92
- renumbered R7 to R10, R6 to R5, R5 to R9
Connections:
- net labels added: BUZZER, EntradaD1, EntradaD2, LED, RX, SalidaD1, Sensor1, Sensor2, TX
- wire segments 73 -> 96
Other:
- note added: "Entradas"
- note added: "Entradas digitales\n multipropósito\n"
- note added: "Indicador luminico"
- note added: "Indicador sonoro\n"
- note added: "PCB:\n- De 1 capa.\n- Transferencia por técnica de planchado.\n- Material: Fibra de vidrio.\n- Color: Azul\n\nEntorno:\n- Temperatura de trabajo: -25ºC a +85ºC\n\nElectrónica:\n- Corriente: 500 miliamperios.\n- Voltaje: 12V DC"
- note added: "Puerto serie para debug"
- note added: "Salida digital\nmultipropósito"
- note added: "Salidas"
- note added: "Sesor de temperatura"
- note removed: "PCB:\n- De 1 capa.\n- Se utilizará técnica de planchado.\n- Material: Fibra de vidrio.\n- Color: Verde.\n\nEntorno:\n- Temperatura de trabajo: -25ºC a +85ºC\n\nElectrónica:\n- Corriente: 500 miliamperios.\n- Voltaje: 12Vts. DC"
