File: SisCoCaf/SisCoCaf.sch (KiCad schematic (older format))
At the start: 20 parts, among them IC1 LPC111X_102, J1 Conn_01x02_Female, J2 Conn_01x02_Female, J3 Conn_01x03_Male, J4 Conn_01x03_Male, J5 Conn_01x01_Male, Q1 BC547, Q2 BC547, U1 LM317_TO39, U2 NRF24L01_Breakout

Commit message: Incorporar pila y jumper
Parts:
- added BT1: Battery_Cell, Battery:BatteryHolder_Keystone_1058_1x2032, symbol Device:Battery_Cell
- added JP1: Jumper_NO_Small, Connector_PinHeader_2.00mm:PinHeader_1x02_P2.00mm_Vertical, symbol Device:Jumper_NO_Small
Changed lines of the file:
@@
 Text Notes 1200 6500 0    79   ~ 0
 PCB:\n- De 1 capa.\n- Se utilizará técnica de planchado.\n- Material: Fibra de vidrio.\n- Color: Verde.\n\nEntorno:\n- Temperatura de trabajo: -25ºC a +85ºC\n\nElectrónica:\n- Corriente: 500 miliamperios.\n- Voltaje: 12Vts. DC
+$Comp
+L Device:Battery_Cell BT1
+U 1 1 5BCA9018
+P 2400 3850
+F 0 "BT1" H 2518 3946 50  0000 L CNN
+F 1 "Battery_Cell" H 2518 3855 50  0000 L CNN
+F 2 "Battery:BatteryHolder_Keystone_1058_1x2032" V 2400 3910 50  0001 C CNN
+F 3 "~" V 2400 3910 50  0001 C CNN
+	1    2400 3850
+	1    0    0    -1
+$EndComp
+$Comp
+L Device:Jumper_NO_Small JP1
+U 1 1 5BCA9157
+P 1750 3850
+F 0 "JP1" H 1750 4035 50  0000 C CNN
+F 1 "Jumper_NO_Small" H 1750 3944 50  0000 C CNN
+F 2 "Connector_PinHeader_2.00mm:PinHeader_1x02_P2.00mm_Vertical" H 1750 3850 50  0001 C CNN
+F 3 "~" H 1750 3850 50  0001 C CNN
+	1    1750 3850
+	1    0    0    -1
+$EndComp
 $EndSCHEMATC

Commit message: Modificando simbolos
Parts:
- removed J4: Conn_01x03_Male, Connector_PinHeader_1.00mm:PinHeader_1x03_P1.00mm_Vertical, symbol Connector:Conn_01x03_Male
- removed JP1: Jumper_NO_Small, Connector_PinHeader_2.00mm:PinHeader_1x02_P2.00mm_Vertical, symbol Device:Jumper_NO_Small
- added J1: Entrada, Connector_JST:JST_XH_B02B-XH-A_1x02_P2.50mm_Vertical, symbol Connector_Generic:Conn_01x02
- added J6: Conn_01x03_Male, Connector_JST:JST_XH_B03B-XH-A_1x03_P2.50mm_Vertical, symbol Connector:Conn_01x03_Male
- added JP1: Jumper, Connector_PinHeader_2.54mm:PinHeader_1x02_P2.54mm_Vertical, symbol Device:Jumper
- added MH1, MH2, MH3, MH4: MountingHole, MountingHole:MountingHole_2.2mm_M2, symbol Mechanical:MountingHole
- added R6, R7: 4k7, Resistor_THT:R_Axial_DIN0204_L3.6mm_D1.6mm_P7.62mm_Horizontal, symbol Device:R
- BT1: footprint Battery:BatteryHolder_Keystone_1058_1x2032 -> Battery:BatteryHolder_Keystone_103_1x20mm
- J2: footprint Connector_PinSocket_1.27mm:PinSocket_1x02_P1.27mm_Vertical -> Connector_PinSocket_2.54mm:PinSocket_1x02_P2.54mm_Vertical
- J4: renamed from J5; footprint Connector_PinHeader_1.00mm:PinHeader_1x02_P1.00mm_Vertical -> Connector_PinHeader_2.54mm:PinHeader_1x01_P2.54mm_Vertical
- J5: renamed from J3; footprint Connector_PinHeader_1.00mm:PinHeader_1x03_P1.00mm_Vertical -> Connector_JST:JST_XH_B03B-XH-A_1x03_P2.50mm_Vertical
- J7: renamed from J1; value Conn_01x02_Female -> Conn_01x02_Male; footprint Connector_PinSocket_1.27mm:PinSocket_1x02_P1.27mm_Vertical -> Connector_JST:JST_XH_B02B-XH-A_1x02_P2.50mm_Vertical
- Q1, Q2: footprint Package_TO_SOT_THT:TO-92_Inline -> Package_TO_SOT_THT:TO-92_HandSolder
- U1: footprint Package_TO_SOT_THT:TO-39-3 -> Package_TO_SOT_THT:TO-220-3_Vertical; symbol Regulator_Linear:LM317_TO39 -> Regulator_Linear:LM317L_TO92
- U2: symbol RF:NRF24L01_Breakout -> RF_TitO:NRF24L01_Breakout
- renumbered R7 to R10, R6 to R5, R5 to R9
Connections:
- net labels added: BUZZER, EntradaD1, EntradaD2, LED, RX, SalidaD1, Sensor1, Sensor2, TX
- wire segments 73 -> 96
Other:
- note added: "Entradas"
- note added: "Entradas digitales\n multipropósito\n"
- note added: "Indicador luminico"
- note added: "Indicador sonoro\n"
- note added: "PCB:\n- De 1 capa.\n- Transferencia por técnica de planchado.\n- Material: Fibra de vidrio.\n- Color: Azul\n\nEntorno:\n- Temperatura de trabajo: -25ºC a +85ºC\n\nElectrónica:\n- Corriente: 500 miliamperios.\n- Voltaje: 12V DC"
- note added: "Puerto serie para debug"
- note added: "Salida digital\nmultipropósito"
- note added: "Salidas"
- note added: "Sesor de temperatura"
- note removed: "PCB:\n- De 1 capa.\n- Se utilizará técnica de planchado.\n- Material: Fibra de vidrio.\n- Color: Verde.\n\nEntorno:\n- Temperatura de trabajo: -25ºC a +85ºC\n\nElectrónica:\n- Corriente: 500 miliamperios.\n- Voltaje: 12Vts. DC"
