File: SisCoCaf/SisCoCaf.sch (KiCad schematic (older format))
At the start: 29 parts, among them IC1 LPC111X_102, J1 Entrada, J2 Conn_01x02_Female, J4 Conn_01x01_Male, J5 Conn_01x03_Male, J6 Conn_01x03_Male, J7 Conn_01x02_Male, Q1 BC547, Q2 BC547, U1 LM317_TO39, U2 NRF24L01_Breakout

Commit message: Versión final.
Realizo correcciones indicadas por profesor.
Parts:
- added C1: 100uf, Capacitor_THT:CP_Radial_D4.0mm_P2.00mm, symbol Device:CP
- added C2: 220uf, Capacitor_THT:CP_Radial_D4.0mm_P2.00mm, symbol Device:CP
- U2: footprint RF_Module:nRF24L01_Breakout -> RF_Module:nRF24L01_Breakout_antena; symbol RF:NRF24L01_Breakout -> RF_TitO:NRF24L01_Breakout
- renumbered J5 to J2, J6 to J3, J7 to J4, J2 to J5, J4 to J6, R8 to R2, R9 to R3, R6 to R4, R7 to R5, R2 to R6, R3 to R7, R4 to R8, R5 to R9
Connections:
- wire segments 96 -> 103
- no-connect marks 13 -> 12
